Commit message: major release: moved to gazebo fortress

File: src/limo_simulation/model/limo_four_diff.xacro (robot description, xacro)
@@ -77,9 +77,11 @@
     </xacro:limo_wheel>
 <gazebo reference="$(arg robot_name)/laser_link">
-    <sensor name="laser" type="ray">
+    <sensor name="laser" type="gpu_lidar">
+      <topic>/$(arg robot_name)/scan</topic>
+      <ignition_frame_id>$(arg robot_name)/laser_link</ignition_frame_id>
       <always_on>true</always_on>
       <visualize>false</visualize>
       <update_rate>8</update_rate>
-      <ray>
+      <lidar>
         <scan>
           <horizontal>
@@ -100,13 +102,5 @@
           <stddev>0.01</stddev>
         </noise>
-      </ray>
-      <plugin name="scan" filename="libgazebo_ros_ray_sensor.so">
-        <ros>
-          <namespace>$(arg robot_name)</namespace>
-          <remapping>~/out:=scan</remapping>
-        </ros>
-        <output_type>sensor_msgs/LaserScan</output_type>
-        <frame_name>$(arg robot_name)/laser_link</frame_name>
-      </plugin>
+      </lidar>
     </sensor>
   </gazebo>

File: src/limo_simulation/model/limo_xacro.xacro (robot description, xacro)
@@ -18,5 +18,5 @@
             </visual>
             <collision>
-              <origin xyz="0 ${wheel_length/2} 0" rpy="1.57 0 0" />
+              <origin xyz="0 0 0" rpy="1.57 0 0" />
               <geometry>
                   <cylinder length="${wheel_length}" radius="${wheel_radius}" />
