Commit message: Multi-robot simulation: n_robots arg, model/controller fixes, rviz and teleop launchers
- gazebo_models_diff.launch.py: n_robots/seed/gui/rviz launch arguments,
  non-overlapping random spawn poses, world -> robot_N/odom static TF,
  generated RViz config. Robots are spawned sequentially because
  gazebo_ros2_control stores its namespace in the global ROS args, which
  put every controller in the last robot's namespace.
- New rviz_models.launch.py (N robots in RViz only, no Gazebo) and
  teleop.launch.py (keyboard teleop of one robot, robot:=robot_N).
- URDF: prefix all links per robot, consistent track (0.172), physical
  inertias, single working IMU, camera frame, laser min range 0.1 m,
  skid-steer wheel friction/contact tuning, removed dead ROS 1 code.
- Controller yaml: real Humble diff_drive_controller parameters.
- Test publishers: robot parameter, missing shebang, clean shutdown.
- README: simulation usage.

Co-Authored-By: Claude Opus 5.5 <noreply@anthropic.com>

File: src/limo_simulation/model/limo_four_diff.xacro (robot description, xacro)
@@ -12,9 +12,10 @@
   <xacro:property name="base_z_size" value="0.1" />
   <xacro:property name="wheelbase" value="0.2"/>
-  <xacro:property name="track" value="0.13"/>
+  <xacro:property name="track" value="0.172"/>
   <xacro:property name="wheel_vertical_offset" value="-0.10" />
   <xacro:property name="base_mass" value="2.1557"/>
   <xacro:property name="wheel_length" value="0.045" />
   <xacro:property name="wheel_radius" value="0.045" />
+  <xacro:property name="wheel_mass" value="0.5" />
   <link name="$(arg robot_name)/base_footprint"/>
   <joint name="$(arg robot_name)/base_joint" type="fixed">
@@ -43,7 +44,8 @@
             <origin xyz="0.0 0.0 0.0" />
             <mass value="${base_mass}" />
-            <inertia ixx="0.24" ixy="0" ixz="0"
-                     iyy="0.96" iyz="0"
-                     izz="0.96" />
+            <!-- solid box inertia -->
+            <inertia ixx="${base_mass/12*(base_y_size**2 + base_z_size**2)}" ixy="0" ixz="0"
+                     iyy="${base_mass/12*(base_x_size**2 + base_z_size**2)}" iyz="0"
+                     izz="${base_mass/12*(base_x_size**2 + base_y_size**2)}" />
         </inertial>
     </link>
@@ -74,84 +76,6 @@
         <origin xyz="${-wheelbase/2} ${-track/2} ${wheel_vertical_offset}" rpy="${M_PI} 0 0" />
     </xacro:limo_wheel>
-    <gazebo reference="imu_link">
-    <gravity>true</gravity>
-    <sensor name="twr_imu" type="imu">
-      <always_on>true</always_on>
-      <update_rate>100</update_rate>
-      <visualize>true</visualize>
-      <imu>
-        <orientation>
-          <x>
-            <noise type="gaussian">
-              <mean>0.0</mean>
-              <stddev>2e-3</stddev>
-            </noise>
-          </x>
-          <y>
-            <noise type="gaussian">
-              <mean>0.0</mean>
-              <stddev>2e-3</stddev>
-            </noise>
-          </y>
-          <z>
-            <noise type="gaussian">
-              <mean>0.0</mean>
-              <stddev>2e-3</stddev>
-            </noise>
-          </z>
-        </orientation>
-        <angular_velocity>
-          <x>
-            <noise type="gaussian">
-              <mean>0.0</mean>
-              <stddev>2e-4</stddev>
-            </noise>
-          </x>
-          <y>
-            <noise type="gaussian">
-              <mean>0.0</mean>
-              <stddev>2e-4</stddev>
-            </noise>
-          </y>
-          <z>
-            <noise type="gaussian">
-              <mean>0.0</mean>
-              <stddev>2e-4</stddev>
-            </noise>
-          </z>
-        </angular_velocity>
-        <linear_acceleration>
-          <x>
-            <noise type="gaussian">
-              <mean>0.0</mean>
-              <stddev>1.7e-2</stddev>
-            </noise>
-          </x>
-          <y>
-            <noise type="gaussian">
-              <mean>0.0</mean>
-              <stddev>1.7e-2</stddev>
-            </noise>
-          </y>
-          <z>
-            <noise type="gaussian">
-              <mean>0.0</mean>
-              <stddev>1.7e-2</stddev>
-            </noise>
-          </z>
-        </linear_acceleration>
-      </imu>
-      <plugin name="$(arg robot_name)_two_wheeled_robot_imu" filename="libgazebo_ros_imu_sensor.so">
-        <initial_orientation_as_reference>false</initial_orientation_as_reference>
-        <frame_name>imu_link</frame_name>
-        <ros>
-          <namespace>/imu</namespace>
-          <remapping>~/out:=data</remapping>
-        </ros>
-      </plugin>
-    </sensor>
-</gazebo>
 <gazebo reference="$(arg robot_name)/laser_link">
-    <sensor name="$(arg robot_name)/laser" type="ray">
+    <sensor name="laser" type="ray">
       <always_on>true</always_on>
       <visualize>false</visualize>
@@ -167,5 +91,5 @@
         </scan>
         <range>
-          <min>0.3</min>
+          <min>0.1</min>
           <max>8.0</max>
           <resolution>0.015</resolution>

File: src/limo_simulation/model/limo_xacro.xacro (robot description, xacro)
@@ -2,9 +2,12 @@
 <robot name="limo_xacro" xmlns:xacro="http://ros.org/wiki/xacro">
     <xacro:macro name="limo_wheel" params="parent_prefix wheel_prefix reflect *joint_pose">
-        <link name="${wheel_prefix}_wheel_link">
+        <link name="$(arg robot_name)/${wheel_prefix}_wheel_link">
             <inertial>
                 <origin xyz="0 0 0" />
-                <mass value="0.5" />
-                <inertia ixx="0.01055" ixy="0" ixz="0" iyy="0.00075" iyz="0" izz="0.01055" />
+                <mass value="${wheel_mass}" />
+                <!-- solid cylinder inertia, axis along y -->
+                <inertia ixx="${wheel_mass*(3*wheel_radius**2 + wheel_length**2)/12}" ixy="0" ixz="0"
+                         iyy="${wheel_mass*wheel_radius**2/2}" iyz="0"
+                         izz="${wheel_mass*(3*wheel_radius**2 + wheel_length**2)/12}" />
             </inertial>
             <visual>
@@ -23,5 +26,5 @@
         <joint name="${wheel_prefix}_wheel" type="continuous">
             <parent link="${parent_prefix}"/>
-            <child link="${wheel_prefix}_wheel_link"/>
+            <child link="$(arg robot_name)/${wheel_prefix}_wheel_link"/>
             <xacro:insert_block name="joint_pose"/>
             <axis xyz="0 ${reflect*1} 0"/>
@@ -45,10 +48,4 @@
                     <cylinder radius="0.02" length="0.01"/>
                 </geometry>
-                <!--<material name='laser_material'>
-                    <ambient>0.1 0.1 0.1 1</ambient>
-                    <diffuse>0.1 0.1 0.2 1</diffuse>
-                    <specular>0 0 0 0</specular>
-                    <emissive>0 0 0 1</emissive>
-                </material>-->
             </visual>
             <collision name='laser_collision'>
@@ -85,10 +82,4 @@
                     <box size="0.02 0.06 0.015"/>
                 </geometry>
-                <!--<material name='depth_camera_material'>
-                    <ambient>0.1 0.1 0.1 1</ambient>
-                    <diffuse>0.1 0.1 0.2 1</diffuse>
-                    <specular>0 0 0 0</specular>
-                    <emissive>0 0 0 1</emissive>
-                </material>-->
             </visual>
             <collision name='depth_camera_collision'>
@@ -104,9 +95,9 @@
             <parent link="${parent_prefix}"/>
         </joint>
-        <link name="depth_link"></link>
+        <link name="$(arg robot_name)/depth_link"></link>
         <joint name="${frame_prefix}_to_camera_joint" type="fixed">
             <origin xyz="0 0 0" rpy="${-M_PI/2} 0 ${-M_PI/2} "/>
             <parent link="${frame_prefix}_link"/>
-            <child link="depth_link"/>
+            <child link="$(arg robot_name)/depth_link"/>
           </joint>
         <gazebo reference="${frame_prefix}_link">
@@ -131,10 +122,4 @@
                     <box size="0.001 0.001 0.001"/>
                 </geometry>
-                <!--<material name='imu_material'>
-                    <ambient>0.1 0.1 0.1 1</ambient>
-                    <diffuse>0.1 0.1 0.2 1</diffuse>
-                    <specular>0 0 0 0</specular>
-                    <emissive>0 0 0 1</emissive>
-                </material>-->
             </visual>
             <collision name='imu_collision'>

Commit message: Multi-robot simulation on Foxy (Gazebo Classic)
Port of the humble multi-robot work (n_robots arg, launch_utils, rviz and
teleop launchers, model/controller fixes), adapted to Foxy:
- spawner.py and positional static_transform_publisher arguments
- per-robot controller yaml with explicit namespaces and robot_N/odom frames
  (no wildcard params or tf_frame_prefix on Foxy)
- unstamped cmd_vel (Foxy teleop_twist_keyboard), /odom remapped per robot
- spawn_delay before the first spawn, absolute sensor topics to work around
  gazebo_ros2_control leaking the previous robot's namespace
- no namespaced xacro include (xacro 2.0.7 bug)
- run.bash: X11 display and GPU access; Dockerfile: rosbridge-suite

Co-Authored-By: Claude Opus 5.5 <noreply@anthropic.com>

File: src/limo_simulation/model/limo_four_diff.xacro (robot description, xacro)
@@ -4,5 +4,5 @@
   <xacro:arg name="namespace" default=""/>
   <xacro:include filename="$(find limo_simulation)/model/limo_xacro.xacro" />
-  <xacro:include filename="$(find limo_simulation)/model/limo_four_diff.gazebo" ns='$(arg namespace)'/>
+  <xacro:include filename="$(find limo_simulation)/model/limo_four_diff.gazebo"/> <!-- no ns: xacro 2.0.7 (Foxy) fails on macro calls in namespaced includes -->
   <!-- Variables -->
   <xacro:property name="M_PI" value="3.14159"/>
@@ -12,9 +12,10 @@
   <xacro:property name="base_z_size" value="0.1" />
   <xacro:property name="wheelbase" value="0.2"/>
-  <xacro:property name="track" value="0.13"/>
+  <xacro:property name="track" value="0.172"/>
   <xacro:property name="wheel_vertical_offset" value="-0.10" />
   <xacro:property name="base_mass" value="2.1557"/>
   <xacro:property name="wheel_length" value="0.045" />
   <xacro:property name="wheel_radius" value="0.045" />
+  <xacro:property name="wheel_mass" value="0.5" />
   <link name="$(arg robot_name)/base_footprint"/>
   <joint name="$(arg robot_name)/base_joint" type="fixed">
@@ -43,7 +44,8 @@
             <origin xyz="0.0 0.0 0.0" />
             <mass value="${base_mass}" />
-            <inertia ixx="0.24" ixy="0" ixz="0"
-                     iyy="0.96" iyz="0"
-                     izz="0.96" />
+            <!-- solid box inertia -->
+            <inertia ixx="${base_mass/12*(base_y_size**2 + base_z_size**2)}" ixy="0" ixz="0"
+                     iyy="${base_mass/12*(base_x_size**2 + base_z_size**2)}" iyz="0"
+                     izz="${base_mass/12*(base_x_size**2 + base_y_size**2)}" />
         </inertial>
     </link>
@@ -74,84 +76,6 @@
         <origin xyz="${-wheelbase/2} ${-track/2} ${wheel_vertical_offset}" rpy="${M_PI} 0 0" />
     </xacro:limo_wheel>
-    <gazebo reference="imu_link">
-    <gravity>true</gravity>
-    <sensor name="twr_imu" type="imu">
-      <always_on>true</always_on>
-      <update_rate>100</update_rate>
-      <visualize>true</visualize>
-      <imu>
-        <orientation>
-          <x>
-            <noise type="gaussian">
-              <mean>0.0</mean>
-              <stddev>2e-3</stddev>
-            </noise>
-          </x>
-          <y>
-            <noise type="gaussian">
-              <mean>0.0</mean>
-              <stddev>2e-3</stddev>
-            </noise>
-          </y>
-          <z>
-            <noise type="gaussian">
-              <mean>0.0</mean>
-              <stddev>2e-3</stddev>
-            </noise>
-          </z>
-        </orientation>
-        <angular_velocity>
-          <x>
-            <noise type="gaussian">
-              <mean>0.0</mean>
-              <stddev>2e-4</stddev>
-            </noise>
-          </x>
-          <y>
-            <noise type="gaussian">
-              <mean>0.0</mean>
-              <stddev>2e-4</stddev>
-            </noise>
-          </y>
-          <z>
-            <noise type="gaussian">
-              <mean>0.0</mean>
-              <stddev>2e-4</stddev>
-            </noise>
-          </z>
-        </angular_velocity>
-        <linear_acceleration>
-          <x>
-            <noise type="gaussian">
-              <mean>0.0</mean>
-              <stddev>1.7e-2</stddev>
-            </noise>
-          </x>
-          <y>
-            <noise type="gaussian">
-              <mean>0.0</mean>
-              <stddev>1.7e-2</stddev>
-            </noise>
-          </y>
-          <z>
-            <noise type="gaussian">
-              <mean>0.0</mean>
-              <stddev>1.7e-2</stddev>
-            </noise>
-          </z>
-        </linear_acceleration>
-      </imu>
-      <plugin name="$(arg robot_name)_two_wheeled_robot_imu" filename="libgazebo_ros_imu_sensor.so">
-        <initial_orientation_as_reference>false</initial_orientation_as_reference>
-        <frame_name>imu_link</frame_name>
-        <ros>
-          <namespace>/imu</namespace>
-          <remapping>~/out:=data</remapping>
-        </ros>
-      </plugin>
-    </sensor>
-</gazebo>
 <gazebo reference="$(arg robot_name)/laser_link">
-    <sensor name="$(arg robot_name)/laser" type="ray">
+    <sensor name="laser" type="ray">
       <always_on>true</always_on>
       <visualize>false</visualize>
@@ -167,5 +91,5 @@
         </scan>
         <range>
-          <min>0.3</min>
+          <min>0.1</min>
           <max>8.0</max>
           <resolution>0.015</resolution>
@@ -180,5 +104,6 @@
         <ros>
           <namespace>$(arg robot_name)</namespace>
-          <remapping>~/out:=scan</remapping>
+          <!-- absolute topic: on Foxy gazebo_ros2_control leaks the previous robot's namespace into later plugins -->
+          <remapping>~/out:=/$(arg robot_name)/scan</remapping>
         </ros>
         <output_type>sensor_msgs/LaserScan</output_type>
